File: ServoSwitch.kicad_pcb (KiCad board)
At the start: 2 copper layers, 42 x 77 mm, 76 parts, among them J1 Conn_01x06_Male, J10 ServoInputSW, J11 ServoOut, J12 ServoInputSW, J13 ServoOut, J14 ServoInputSW, J15 ServoOut, J16 ServoInputSW, J17 ServoOut, J18 ServoInputSW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

Commit message: Add licence
Other:
- board text added: "SPDX-FileCopyrightText: 2023 Antonios Vamporakis <ant@anttronics.com> SPDX-License-Identifier: CERN-OHL-W-2.0+ You may redistribute and modify this documentation and make products using it under the terms of the CERN-OHL-W v2 (https:/cern.ch/cern-ohl). This documentation is distributed WITHOUT ANY EXPRESS OR IMPLIED WARRANTY, INCLUDING OF MERCHANTABILITY, SATISFACTORY QUALITY AND FITNESS FOR A PA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"
Changed lines of the file:
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@@
   )
   (paper "A4")
+  (title_block
+    (title "ServoSwitch")
+    (date "2023-12-20")
+    (rev "0.1")
+    (company "AntTronics")
+  )
   (layers
     (0 "F.Cu" signal)
@@
     (effects (font (size 1.5 1.5) (thickness 0.3)))
   )
+  (gr_text "SPDX-FileCopyrightText: 2023 Antonios Vamporakis <ant@anttronics.com>\nSPDX-License-Identifier: CERN-OHL-W-2.0+\n\nYou may redistribute and modify this documentation and make products\nusing it under the terms of the CERN-OHL-W v2 (https:/cern.ch/cern-ohl).\nThis documentation is distributed WITHOUT ANY EXPRESS OR IMPLIED\nWARRANTY, INCLUDING OF MERCHANTABILITY, SATISFACTORY QUALITY\nAND FITNESS FOR A PARTICULAR PURPOSE. Please see the CERN-OHL-W v2\nfor applicable conditions.\n\nSource location: https://github.com/anttronics/SolarTrackerSensor\n\nAs per CERN-OHL-W v2 section 4.1, should You produce hardware based on\nthese sources, You must maintain the Source Location visible on the\nexternal case of the ServoSwitch or other product you make using\nthis documentation.\n" (at 236.5 177) (layer "Cmts.User")
+    (effects (font (size 0.8 0.8) (thickness 0.15)) (justify left))
+  )
   (segment (start 183.75 58.29) (end 184.55 58.29) (width 0.3) (layer "F.Cu") (net 1))
