File: ServoSwitch.kicad_sch (KiCad schematic)
At the start: 42 parts, among them J1 Conn_01x06_Male, J2 TagConnect, J3 6V-15V IN, J4 USB_C_Receptacle_USB2.0, J5 5V IN, SW1 Push Button NO 12mm SMD, SW2 Push Button NO 12mm SMD, U1 STM32F030C8T6TR, U2 EA8212FT6R, U3 AMS1117-3.3

Commit message: Add licence
Other:
- note added: "SPDX-FileCopyrightText: 2023 Antonios Vamporakis <ant@anttronics.com> SPDX-License-Identifier: CERN-OHL-W-2.0+ You may redistribute and modify this documentation and make products using it under the terms of the CERN-OHL-W v2 (https:/cern.ch/cern-ohl). This documentation is distributed WITHOUT ANY EXPRESS OR IMPLIED WARRANTY, INCLUDING OF MERCHANTABILITY, SATISFACTORY QUALITY AND FITNESS FOR A PA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"
- company: (none) -> AntTronics
- title: (none) -> ServoSwitch
Changed lines of the file:
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@@
 (kicad_sch (version 20211123) (generator eeschema)
   (paper "A4")
+  (title_block
+    (title "ServoSwitch")
+    (date "2023-12-20")
+    (rev "0.1")
+    (company "AntTronics")
+  )
   (junction (at 171.45 133.985) (diameter 0) (color 0 0 0 0)
   )
@@
     (effects (font (size 1.27 1.27)) (justify left bottom))
   )
+  (text "SPDX-FileCopyrightText: 2023 Antonios Vamporakis <ant@anttronics.com>\nSPDX-License-Identifier: CERN-OHL-W-2.0+\n\nYou may redistribute and modify this documentation and make products\nusing it under the terms of the CERN-OHL-W v2 (https:/cern.ch/cern-ohl).\nThis documentation is distributed WITHOUT ANY EXPRESS OR IMPLIED\nWARRANTY, INCLUDING OF MERCHANTABILITY, SATISFACTORY QUALITY\nAND FITNESS FOR A PARTICULAR PURPOSE. Please see the CERN-OHL-W v2\nfor applicable conditions.\n\nSource location: https://github.com/anttronics/SolarTrackerSensor\n\nAs per CERN-OHL-W v2 section 4.1, should You produce hardware based on\nthese sources, You must maintain the Source Location visible on the\nexternal case of the ServoSwitch or other product you make using\nthis documentation.\n"
+    (at 236.22 186.69 0)
+    (effects (font (size 0.8 0.8)) (justify left bottom))
+  )
   (text "6V - 18V" (at 180.975 113.665 0)
